Commit message: update endeffector joint for moveit

File: config/ur10_with_gripper.urdf.xacro (robot description, xacro)
@@ -1,10 +1,617 @@
-<?xml version="1.0"?>
-<robot xmlns:xacro="http://www.ros.org/wiki/xacro" name="ur10_with_gripper">
-    <xacro:arg name="initial_positions_file" default="$(find moveit_ur10)/config/initial_positions.yaml" />
-    <xacro:arg name="ros2_control_hardware_type" default="mock_components" />
-    <!-- Import ur10_with_gripper urdf file -->
-    <xacro:include filename="ur10_with_gripper_sim.urdf" />
-    <!-- Import control_xacro -->
-    <xacro:include filename="ur10.ros2_control.xacro" />
-    <xacro:ur10_ros2_control name="FakeSystem" initial_positions_file="$(arg initial_positions_file)" ros2_control_hardware_type="$(arg ros2_control_hardware_type)"/>
+<?xml version="1.0" ?>
+<!-- =================================================================================== -->
+<!-- |    This document was autogenerated by xacro from ur_description/urdf/ur10_with_gripper.xacro | -->
+<!-- |    EDITING THIS FILE BY HAND IS NOT RECOMMENDED                                 | -->
+<!-- =================================================================================== -->
+<robot name="ur10_with_gripper">
+  <!--
+    Base UR robot series xacro macro.
+    NOTE this is NOT a URDF. It cannot directly be loaded by consumers
+    expecting a flattened '.urdf' file. See the top-level '.xacro' for that
+    (but note that .xacro must still be processed by the xacro command).
+    This file models the base kinematic chain of a UR robot, which then gets
+    parameterised by various configuration files to convert it into a UR3(e),
+    UR5(e), UR10(e) or UR16e.
+    NOTE the default kinematic parameters (i.e., link lengths, frame locations,
+    offsets, etc) do not correspond to any particular robot. They are defaults
+    only. There WILL be non-zero offsets between the Forward Kinematics results
+    in TF (i.e., robot_state_publisher) and the values reported by the Teach
+    Pendant.
+    For accurate (and robot-specific) transforms, the 'kinematics_parameters_file'
+    parameter MUST point to a .yaml file containing the appropriate values for
+    the targeted robot.
+    If using the UniversalRobots/Universal_Robots_ROS_Driver, follow the steps
+    described in the readme of that repository to extract the kinematic
+    calibration from the controller and generate the required .yaml file.
+    Main author of the migration to yaml configs Ludovic Delval.
+    Contributors to previous versions (in no particular order)
+     - Denis Stogl
+     - Lovro Ivanov
+     - Felix Messmer
+     - Kelsey Hawkins
+     - Wim Meeussen
+     - Shaun Edwards
+     - Nadia Hammoudeh Garcia
+     - Dave Hershberger
+     - G. vd. Hoorn
+     - Philip Long
+     - Dave Coleman
+     - Miguel Prada
+     - Mathias Luedtke
+     - Marcel Schnirring
+     - Felix von Drigalski
+     - Felix Exner
+     - Jimmy Da Silva
+     - Ajit Krisshna N L
+     - Muhammad Asif Rana
+  -->
+  <!--
+    NOTE the macro defined in this file is NOT part of the public API of this
+          package. Users CANNOT rely on this file being available, or stored in
+          this location. Nor can they rely on the existence of the macro.
+  -->
+  <!-- Create world link -->
+  <link name="world"/>
+  <ros2_control name="ur10" type="system">
+    <hardware>
+      <plugin>mock_components/GenericSystem</plugin>
+      <param name="robot_ip">0.0.0.0</param>
+      <param name="script_filename">to_be_filled_by_ur_robot_driver</param>
+      <param name="output_recipe_filename">to_be_filled_by_ur_robot_driver</param>
+      <param name="input_recipe_filename">to_be_filled_by_ur_robot_driver</param>
+      <param name="headless_mode">False</param>
+      <param name="reverse_port">50001</param>
+      <param name="script_sender_port">50002</param>
+      <param name="reverse_ip">0.0.0.0</param>
+      <param name="script_command_port">50004</param>
+      <param name="trajectory_port">50003</param>
+      <param name="tf_prefix"></param>
+      <param name="non_blocking_read">True</param>
+      <param name="servoj_gain">2000</param>
+      <param name="servoj_lookahead_time">0.03</param>
+      <param name="use_tool_communication">False</param>
+      <param name="kinematics/hash">calib_17227329492635474227</param>
+      <param name="tool_voltage">0</param>
+      <param name="tool_parity">0</param>
+      <param name="tool_baud_rate">115200</param>
+      <param name="tool_stop_bits">1</param>
+      <param name="tool_rx_idle_chars">1.5</param>
+      <param name="tool_tx_idle_chars">3.5</param>
+      <param name="tool_device_name">/tmp/ttyUR</param>
+      <param name="tool_tcp_port">54321</param>
+      <param name="keep_alive_count">2</param>
+    </hardware>
+    <joint name="shoulder_pan_joint">
+      <command_interface name="position"/>
+      <command_interface name="velocity"/>
+      <state_interface name="position">
+        <!-- initial position for the FakeSystem and simulation -->
+        <param name="initial_value">0.0</param>
+      </state_interface>
+      <state_interface name="velocity"/>
+      <state_interface name="effort"/>
+    </joint>
+    <joint name="shoulder_lift_joint">
+      <command_interface name="position"/>
+      <command_interface name="velocity"/>
+      <state_interface name="position">
+        <!-- initial position for the FakeSystem and simulation -->
+        <param name="initial_value">-1.57</param>
+      </state_interface>
+      <state_interface name="velocity"/>
+      <state_interface name="effort"/>
+    </joint>
+    <joint name="elbow_joint">
+      <command_interface name="position"/>
+      <command_interface name="velocity"/>
+      <state_interface name="position">
+        <!-- initial position for the FakeSystem and simulation -->
+        <param name="initial_value">0.0</param>
+      </state_interface>
+      <state_interface name="velocity"/>
+      <state_interface name="effort"/>
+    </joint>
+    <joint name="wrist_1_joint">
+      <command_interface name="position"/>
+      <command_interface name="velocity"/>
+      <state_interface name="position">
+        <!-- initial position for the FakeSystem and simulation -->
+        <param name="initial_value">-1.57</param>
+      </state_interface>
+      <state_interface name="velocity"/>
+      <state_interface name="effort"/>
+    </joint>
+    <joint name="wrist_2_joint">
+      <command_interface name="position"/>
+      <command_interface name="velocity"/>
+      <state_interface name="position">
+        <!-- initial position for the FakeSystem and simulation -->
+        <param name="initial_value">0.0</param>
+      </state_interface>
+      <state_interface name="velocity"/>
+      <state_interface name="effort"/>
+    </joint>
+    <joint name="wrist_3_joint">
+      <command_interface name="position"/>
+      <command_interface name="velocity"/>
+      <state_interface name="position">
+        <!-- initial position for the FakeSystem and simulation -->
+        <param name="initial_value">0.0</param>
+      </state_interface>
+      <state_interface name="velocity"/>
+      <state_interface name="effort"/>
+    </joint>
+    <sensor name="tcp_fts_sensor">
+      <state_interface name="force.x"/>
+      <state_interface name="force.y"/>
+      <state_interface name="force.z"/>
+      <state_interface name="torque.x"/>
+      <state_interface name="torque.y"/>
+      <state_interface name="torque.z"/>
+    </sensor>
+    <sensor name="tcp_pose">
+      <state_interface name="position.x"/>
+      <state_interface name="position.y"/>
+      <state_interface name="position.z"/>
+      <state_interface name="orientation.x"/>
+      <state_interface name="orientation.y"/>
+      <state_interface name="orientation.z"/>
+      <state_interface name="orientation.w"/>
+    </sensor>
+    <!-- NOTE The following are joints used only for testing with fake hardware and will change in the future -->
+    <gpio name="speed_scaling">
+      <state_interface name="speed_scaling_factor"/>
+      <param name="initial_speed_scaling_factor">1</param>
+      <command_interface name="target_speed_fraction_cmd"/>
+      <command_interface name="target_speed_fraction_async_success"/>
+    </gpio>
+    <gpio name="gpio">
+      <command_interface name="standard_digital_output_cmd_0"/>
+      <command_interface name="standard_digital_output_cmd_1"/>
+      <command_interface name="standard_digital_output_cmd_2"/>
+      <command_interface name="standard_digital_output_cmd_3"/>
+      <command_interface name="standard_digital_output_cmd_4"/>
+      <command_interface name="standard_digital_output_cmd_5"/>
+      <command_interface name="standard_digital_output_cmd_6"/>
+      <command_interface name="standard_digital_output_cmd_7"/>
+      <command_interface name="standard_digital_output_cmd_8"/>
+      <command_interface name="standard_digital_output_cmd_9"/>
+      <command_interface name="standard_digital_output_cmd_10"/>
+      <command_interface name="standard_digital_output_cmd_11"/>
+      <command_interface name="standard_digital_output_cmd_12"/>
+      <command_interface name="standard_digital_output_cmd_13"/>
+      <command_interface name="standard_digital_output_cmd_14"/>
+      <command_interface name="standard_digital_output_cmd_15"/>
+      <command_interface name="standard_digital_output_cmd_16"/>
+      <command_interface name="standard_digital_output_cmd_17"/>
+      <command_interface name="standard_analog_output_cmd_0"/>
+      <command_interface name="standard_analog_output_cmd_1"/>
+      <command_interface name="analog_output_domain_cmd"/>
+      <command_interface name="tool_voltage_cmd"/>
+      <command_interface name="io_async_success"/>
+      <state_interface name="digital_output_0"/>
+      <state_interface name="digital_output_1"/>
+      <state_interface name="digital_output_2"/>
+      <state_interface name="digital_output_3"/>
+      <state_interface name="digital_output_4"/>
+      <state_interface name="digital_output_5"/>
+      <state_interface name="digital_output_6"/>
+      <state_interface name="digital_output_7"/>
+      <state_interface name="digital_output_8"/>
+      <state_interface name="digital_output_9"/>
+      <state_interface name="digital_output_10"/>
+      <state_interface name="digital_output_11"/>
+      <state_interface name="digital_output_12"/>
+      <state_interface name="digital_output_13"/>
+      <state_interface name="digital_output_14"/>
+      <state_interface name="digital_output_15"/>
+      <state_interface name="digital_output_16"/>
+      <state_interface name="digital_output_17"/>
+      <state_interface name="digital_input_0"/>
+      <state_interface name="digital_input_1"/>
+      <state_interface name="digital_input_2"/>
+      <state_interface name="digital_input_3"/>
+      <state_interface name="digital_input_4"/>
+      <state_interface name="digital_input_5"/>
+      <state_interface name="digital_input_6"/>
+      <state_interface name="digital_input_7"/>
+      <state_interface name="digital_input_8"/>
+      <state_interface name="digital_input_9"/>
+      <state_interface name="digital_input_10"/>
+      <state_interface name="digital_input_11"/>
+      <state_interface name="digital_input_12"/>
+      <state_interface name="digital_input_13"/>
+      <state_interface name="digital_input_14"/>
+      <state_interface name="digital_input_15"/>
+      <state_interface name="digital_input_16"/>
+      <state_interface name="digital_input_17"/>
+      <state_interface name="standard_analog_output_0"/>
+      <state_interface name="standard_analog_output_1"/>
+      <state_interface name="standard_analog_input_0"/>
+      <state_interface name="standard_analog_input_1"/>
+      <state_interface name="analog_io_type_0"/>
+      <state_interface name="analog_io_type_1"/>
+      <state_interface name="analog_io_type_2"/>
+      <state_interface name="analog_io_type_3"/>
+      <state_interface name="tool_mode"/>
+      <state_interface name="tool_output_voltage"/>
+      <state_interface name="tool_output_current"/>
+      <state_interface name="tool_temperature"/>
+      <state_interface name="tool_analog_input_0"/>
+      <state_interface name="tool_analog_input_1"/>
+      <state_interface name="tool_analog_input_type_0"/>
+      <state_interface name="tool_analog_input_type_1"/>
+      <state_interface name="robot_mode"/>
+      <state_interface name="robot_status_bit_0"/>
+      <state_interface name="robot_status_bit_1"/>
+      <state_interface name="robot_status_bit_2"/>
+      <state_interface name="robot_status_bit_3"/>
+      <state_interface name="safety_mode"/>
+      <state_interface name="safety_status_bit_0"/>
+      <state_interface name="safety_status_bit_1"/>
+      <state_interface name="safety_status_bit_2"/>
+      <state_interface name="safety_status_bit_3"/>
+      <state_interface name="safety_status_bit_4"/>
+      <state_interface name="safety_status_bit_5"/>
+      <state_interface name="safety_status_bit_6"/>
+      <state_interface name="safety_status_bit_7"/>
+      <state_interface name="safety_status_bit_8"/>
+      <state_interface name="safety_status_bit_9"/>
+      <state_interface name="safety_status_bit_10"/>
+      <state_interface name="program_running"/>
+    </gpio>
+    <gpio name="payload">
+      <command_interface name="mass"/>
+      <command_interface name="cog.x"/>
+      <command_interface name="cog.y"/>
+      <command_interface name="cog.z"/>
+      <command_interface name="payload_async_success"/>
+    </gpio>
+    <gpio name="resend_robot_program">
+      <command_interface name="resend_robot_program_cmd"/>
+      <command_interface name="resend_robot_program_async_success"/>
+    </gpio>
+    <gpio name="hand_back_control">
+      <command_interface name="hand_back_control_cmd"/>
+      <command_interface name="hand_back_control_async_success"/>
+    </gpio>
+    <gpio name="zero_ftsensor">
+      <command_interface name="zero_ftsensor_cmd"/>
+      <command_interface name="zero_ftsensor_async_success"/>
+    </gpio>
+    <gpio name="freedrive_mode">
+      <command_interface name="async_success"/>
+      <command_interface name="enable"/>
+      <command_interface name="abort"/>
+    </gpio>
+    <gpio name="tool_contact">
+      <command_interface name="tool_contact_set_state"/>
+      <state_interface name="tool_contact_result"/>
+      <state_interface name="tool_contact_state"/>
+    </gpio>
+    <gpio name="system_interface">
+      <state_interface name="initialized"/>
+    </gpio>
+    <gpio name="force_mode">
+      <command_interface name="task_frame_x"/>
+      <command_interface name="task_frame_y"/>
+      <command_interface name="task_frame_z"/>
+      <command_interface name="task_frame_rx"/>
+      <command_interface name="task_frame_ry"/>
+      <command_interface name="task_frame_rz"/>
+      <command_interface name="selection_vector_x"/>
+      <command_interface name="selection_vector_y"/>
+      <command_interface name="selection_vector_z"/>
+      <command_interface name="selection_vector_rx"/>
+      <command_interface name="selection_vector_ry"/>
+      <command_interface name="selection_vector_rz"/>
+      <command_interface name="wrench_x"/>
+      <command_interface name="wrench_y"/>
+      <command_interface name="wrench_z"/>
+      <command_interface name="wrench_rx"/>
+      <command_interface name="wrench_ry"/>
+      <command_interface name="wrench_rz"/>
+      <command_interface name="limits_x"/>
+      <command_interface name="limits_y"/>
+      <command_interface name="limits_z"/>
+      <command_interface name="limits_rx"/>
+      <command_interface name="limits_ry"/>
+      <command_interface name="limits_rz"/>
+      <command_interface name="type"/>
+      <command_interface name="damping"/>
+      <command_interface name="gain_scaling"/>
+      <command_interface name="disable_cmd"/>
+      <command_interface name="force_mode_async_success"/>
+    </gpio>
+    <gpio name="trajectory_passthrough">
+      <command_interface name="setpoint_positions_0"/>
+      <command_interface name="setpoint_positions_1"/>
+      <command_interface name="setpoint_positions_2"/>
+      <command_interface name="setpoint_positions_3"/>
+      <command_interface name="setpoint_positions_4"/>
+      <command_interface name="setpoint_positions_5"/>
+      <command_interface name="setpoint_velocities_0"/>
+      <command_interface name="setpoint_velocities_1"/>
+      <command_interface name="setpoint_velocities_2"/>
+      <command_interface name="setpoint_velocities_3"/>
+      <command_interface name="setpoint_velocities_4"/>
+      <command_interface name="setpoint_velocities_5"/>
+      <command_interface name="setpoint_accelerations_0"/>
+      <command_interface name="setpoint_accelerations_1"/>
+      <command_interface name="setpoint_accelerations_2"/>
+      <command_interface name="setpoint_accelerations_3"/>
+      <command_interface name="setpoint_accelerations_4"/>
+      <command_interface name="setpoint_accelerations_5"/>
+      <command_interface name="transfer_state"/>
+      <command_interface name="time_from_start"/>
+      <command_interface name="abort"/>
+    </gpio>
+    <gpio name="get_robot_software_version">
+      <state_interface name="get_version_major"/>
+      <state_interface name="get_version_minor"/>
+      <state_interface name="get_version_build"/>
+      <state_interface name="get_version_bugfix"/>
+    </gpio>
+  </ros2_control>
+  <!-- Add URDF transmission elements (for ros_control) -->
+  <!--<xacro:ur_arm_transmission prefix="${prefix}" hw_interface="${transmission_hw_interface}" />-->
+  <!-- Placeholder for ros2_control transmission which don't yet exist -->
+  <!-- links -  main serial chain -->
+  <link name="base_link"/>
+  <link name="base_link_inertia">
+    <visual>
+      <origin rpy="0 0 3.141592653589793" xyz="0 0 0"/>
+      <geometry>
+        <mesh filename="package://ur_description/meshes/ur10/visual/base.dae"/>
+      </geometry>
+    </visual>
+    <collision>
+      <origin rpy="0 0 3.141592653589793" xyz="0 0 0"/>
+      <geometry>
+        <mesh filename="package://ur_description/meshes/ur10/collision/base.stl"/>
+      </geometry>
+    </collision>
+    <inertial>
+      <mass value="4.0"/>
+      <origin rpy="0 0 0" xyz="0 0 0"/>
+      <inertia ixx="0.0061063308908" ixy="0.0" ixz="0.0" iyy="0.0061063308908" iyz="0.0" izz="0.01125"/>
+    </inertial>
+  </link>
+  <link name="shoulder_link">
+    <visual>
+      <origin rpy="0 0 3.141592653589793" xyz="0 0 0"/>
+      <geometry>
+        <mesh filename="package://ur_description/meshes/ur10/visual/shoulder.dae"/>
+      </geometry>
+    </visual>
+    <collision>
+      <origin rpy="0 0 3.141592653589793" xyz="0 0 0"/>
+      <geometry>
+        <mesh filename="package://ur_description/meshes/ur10/collision/shoulder.stl"/>
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
File: config/ur10_with_gripper_isaac.urdf.xacro (robot description, xacro)
@@ -215,10 +215,10 @@
         <child link="tool0"/>
     </joint>
-    <!-- Base link of the gripper -->
+    <!-- Base link of the gripper with a cylinder geometry -> length of custom gripper -->
     <link name="gripper_base">
         <visual>
-            <origin rpy="0 0 0" xyz="0 0 0.05"/>
-            <geometry>
-                <cylinder length="0.1" radius="0.03"/>
+            <origin rpy="0 0 0" xyz="0 0 0.0"/>
+            <geometry>
+                <cylinder length="0.2" radius="0.03"/>
             </geometry>
             <material name="grey">
@@ -239,4 +239,16 @@
         <origin rpy="0 0 0" xyz="0 0 0"/>
     </joint>
+    <!-- Virtual tip frame for MoveIt interactive marker -->
+    <link name="moveit_eef">
+        <visual>
+            <origin rpy="0 0 0" xyz="0 0 0"/>
+        </visual>
+    </link>
+    <!-- offset of planning frame from gripper base -->
+    <joint name="moveit_eef_joint" type="fixed">
+        <parent link="gripper_base"/>
+        <child link="moveit_eef"/>
+        <origin rpy="0 0 0" xyz="0 0 0.1"/>
+    </joint>
     <!-- Import control_xacro for Isaac -->
     <xacro:include filename="ur10.ros2_control.xacro" />
